File: kinesis_adv2.kicad_pcb (KiCad board)
At the start: 16 copper layers, 122 x 86 mm, 17 parts, among them U1 C-TEENSY++

Commit message: fix M6 mounting hole
Signed-off-by: Antony Pavlov <antonynpavlov@gmail.com>
Parts:
- @HOLE0: value (none) -> MountingHole_6.4mm_M6; footprint (none) -> MountingHole:MountingHole_6.4mm_M6
Changed lines of the file:
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@@
     (pad P$12 thru_hole circle (at 6.25 -1.65) (size 1.5112 1.5112) (drill 0.8) (layers *.Cu *.Mask))
   )
-  (module "" (layer Top)
+  (module MountingHole:MountingHole_6.4mm_M6 (layer Top)
     (at 148.5011 86.5036)
     (fp_text reference @HOLE0 (at 0 0) (layer F.SilkS) hide
       (effects (font (size 1.524 1.524) (thickness 0.15)))
     )
-    (fp_text value "" (at 0 0) (layer F.SilkS)
+    (fp_text value MountingHole_6.4mm_M6 (at 0 7.4) (layer F.Fab)
       (effects (font (size 1.524 1.524) (thickness 0.15)))
     )
-    (pad "" np_thru_hole circle (at 0 0) (size 6.4 6.4) (drill 6.4) (layers *.Cu))
+    (pad 1 np_thru_hole circle (at 0 0) (size 6.4 6.4) (drill 6.4) (layers *.Cu *.Mask))
   )
   (module TEENSY++ (layer Top)
